File: load.kicad_pcb (KiCad board)
At the start: 2 copper layers, 28 parts, among them J1 Load +, J2 Load -, Q1 IRFZ44N, Q2 IRFZ44N, Q3 IRFZ44N, Q4 IRFZ44N, U1 LM358, U2 LM7805_TO220, U3 MCP1525-TO

Commit message: almost
Parts:
- added C10: 10n, Capacitor_SMD:C_0805_2012Metric_Pad1.15x1.40mm_HandSolder, B.Cu at (82.5, 187.3)
- added C11: 100n, Capacitor_SMD:C_0805_2012Metric_Pad1.15x1.40mm_HandSolder, B.Cu at (98.8, 153.7)
- added C12: 100n, Capacitor_SMD:C_0805_2012Metric_Pad1.15x1.40mm_HandSolder, B.Cu at (98.8, 189.2)
- added C8: 10n, Capacitor_SMD:C_0805_2012Metric_Pad1.15x1.40mm_HandSolder, B.Cu at (82.6, 169.5)
- added C9: 10n, Capacitor_SMD:C_0805_2012Metric_Pad1.15x1.40mm_HandSolder, B.Cu at (82.5, 151.8)
- added R12: 100, Resistor_SMD:R_0805_2012Metric_Pad1.15x1.40mm_HandSolder, B.Cu at (90.4, 191.8)
- added R13: 10k, Resistor_SMD:R_0805_2012Metric_Pad1.15x1.40mm_HandSolder, B.Cu at (98.8, 129.5)
- added R14: 10k, Resistor_SMD:R_0805_2012Metric_Pad1.15x1.40mm_HandSolder, B.Cu at (98.7, 165.1)
- added R15: 10k, Resistor_SMD:R_0805_2012Metric_Pad1.15x1.40mm_HandSolder, B.Cu at (98.8, 147.3)
- added R16: 10k, Resistor_SMD:R_0805_2012Metric_Pad1.15x1.40mm_HandSolder, B.Cu at (98.8, 182.9)
- added R17: 0.1, Resistor_THT:R_Axial_DIN0922_L20.0mm_D9.0mm_P30.48mm_Horizontal, F.Cu at (106.7, 132.1)
- added R18: 0.1, Resistor_THT:R_Axial_DIN0922_L20.0mm_D9.0mm_P30.48mm_Horizontal, F.Cu at (106.7, 167.6)
- added R19: 0.1, Resistor_THT:R_Axial_DIN0922_L20.0mm_D9.0mm_P30.48mm_Horizontal, F.Cu at (106.7, 149.9)
- added R20: 0.1, Resistor_THT:R_Axial_DIN0922_L20.0mm_D9.0mm_P30.48mm_Horizontal, F.Cu at (106.7, 185.4)
- added R21: 10k, Resistor_SMD:R_0805_2012Metric_Pad1.15x1.40mm_HandSolder, B.Cu at (98.8, 132.7)
- added R22: 10k, Resistor_SMD:R_0805_2012Metric_Pad1.15x1.40mm_HandSolder, B.Cu at (98.8, 168.3)
- added R23: 10k, Resistor_SMD:R_0805_2012Metric_Pad1.15x1.40mm_HandSolder, B.Cu at (98.8, 150.5)
- added R24: 10k, Resistor_SMD:R_0805_2012Metric_Pad1.15x1.40mm_HandSolder, B.Cu at (98.8, 186.1)
- added R25: 10k, Resistor_SMD:R_0805_2012Metric_Pad1.15x1.40mm_HandSolder, B.Cu at (98.8, 126.4)
- added R26: 10k, Resistor_SMD:R_0805_2012Metric_Pad1.15x1.40mm_HandSolder, B.Cu at (98.7, 161.9)
- added R27: 10k, Resistor_SMD:R_0805_2012Metric_Pad1.15x1.40mm_HandSolder, B.Cu at (98.8, 144.1)
- added R28: 10k, Resistor_SMD:R_0805_2012Metric_Pad1.15x1.40mm_HandSolder, B.Cu at (98.8, 179.7)
- added R29: 10k, Resistor_SMD:R_0805_2012Metric_Pad1.15x1.40mm_HandSolder, B.Cu at (91.2, 127.0)
- added R30: 10k, Resistor_SMD:R_0805_2012Metric_Pad1.15x1.40mm_HandSolder, B.Cu at (91.2, 162.6)
- added R31: 10k, Resistor_SMD:R_0805_2012Metric_Pad1.15x1.40mm_HandSolder, B.Cu at (91.2, 144.8)
- added R32: 10k, Resistor_SMD:R_0805_2012Metric_Pad1.15x1.40mm_HandSolder, B.Cu at (91.2, 180.3)
- added R33: 30k, Resistor_SMD:R_0805_2012Metric_Pad1.15x1.40mm_HandSolder, B.Cu at (54.4, 188.0)
- added R34: 10k, Resistor_SMD:R_0805_2012Metric_Pad1.15x1.40mm_HandSolder, B.Cu at (59.9, 188.0)
- added U4: LM358, Package_SO:SO-8_5.3x6.2mm_P1.27mm, B.Cu at (90.2, 168.3)
- added U5: LM358, Package_SO:SO-8_5.3x6.2mm_P1.27mm, B.Cu at (90.2, 150.5)
- added U6: LM358, Package_SO:SO-8_5.3x6.2mm_P1.27mm, B.Cu at (90.2, 186.1)
- C1: footprint Capacitor_THT:CP_Radial_D4.0mm_P2.00mm -> Capacitor_SMD:C_0805_2012Metric_Pad1.15x1.40mm_HandSolder; moved to B.Cu
- C2, C3, C4, C5, C6, C7: footprint Capacitor_THT:C_Disc_D5.0mm_W2.5mm_P2.50mm -> Capacitor_SMD:C_0805_2012Metric_Pad1.15x1.40mm_HandSolder; moved to B.Cu
- Q1, Q2, Q3, Q4: value IRFZ44N -> Q_NMOS_GDS
- R1, R2, R3, R4, R9: footprint Resistor_THT:R_Axial_DIN0207_L6.3mm_D2.5mm_P2.54mm_Vertical -> Resistor_SMD:R_0805_2012Metric_Pad1.15x1.40mm_HandSolder; moved to B.Cu
- R10, R11: value 10k -> 100; footprint Resistor_THT:R_Axial_DIN0207_L6.3mm_D2.5mm_P2.54mm_Vertical -> Resistor_SMD:R_0805_2012Metric_Pad1.15x1.40mm_HandSolder; moved to B.Cu
- R5, R6, R8: footprint Resistor_THT:R_Axial_DIN0207_L6.3mm_D2.5mm_P2.54mm_Vertical -> Resistor_SMD:R_0805_2012Metric_Pad1.15x1.40mm_HandSolder
- R7: footprint Resistor_THT:R_Axial_DIN0207_L6.3mm_D2.5mm_P10.16mm_Horizontal -> Resistor_SMD:R_0805_2012Metric_Pad1.15x1.40mm_HandSolder
- RV1: footprint Potentiometer_THT:Potentiometer_Bourns_3266W_Vertical -> Potentiometer_THT:Potentiometer_Alps_RK097_Single_Horizontal
- U1: footprint Package_DIP:DIP-8_W7.62mm -> Package_SO:SO-8_5.3x6.2mm_P1.27mm; moved to B.Cu
- moved J2 116.6 mm to (55.9, 132.1)
- moved Q4 109.3 mm to (116.8, 188.0)
- moved R4 107.6 mm to (86.4, 192.8), turned to 90 degrees
- moved C6 95.9 mm to (59.9, 180.3), turned to 0 degrees
- moved R8 95.4 mm to (112.8, 188.0), turned to 0 degrees
- moved R2 94.2 mm to (86.4, 175.0), turned to 90 degrees
- moved C5 93.2 mm to (54.9, 167.6)
- moved U3 93.0 mm to (53.3, 163.8)
- moved Q2 92.0 mm to (116.8, 170.2)
- moved RV1 90.4 mm to (55.9, 177.8), turned to 180 degrees
- moved R11 89.6 mm to (90.4, 156.2), turned to 0 degrees
- moved C4 84.0 mm to (58.4, 156.8)
- moved U2 77.0 mm to (53.3, 153.7)
- moved R3 75.9 mm to (86.4, 157.2), turned to 90 degrees
- moved R10 75.4 mm to (90.4, 174.0), turned to 0 degrees
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Connections:
- Q1 pad 2: VCC -> VDD
- Q2 pad 2: VCC -> VDD
- Q2 pad 3: Net-(Q1-Pad3) -> Net-(Q2-Pad3)
- Q3 pad 2: VCC -> VDD
- Q3 pad 3: Net-(Q1-Pad3) -> Net-(Q3-Pad3)
- Q4 pad 2: VCC -> VDD
- Q4 pad 3: Net-(Q1-Pad3) -> Net-(Q4-Pad3)
- R10 pad 1: GND -> Net-(C8-Pad2)
- R10 pad 2: Net-(C7-Pad1) -> Net-(R10-Pad2)
- R11 pad 1: GND -> Net-(C9-Pad2)
- R11 pad 2: Net-(Q1-Pad3) -> Net-(R11-Pad2)
- R2 pad 2: Net-(C7-Pad1) -> Net-(C8-Pad1)
- R3 pad 2: Net-(C7-Pad1) -> Net-(C9-Pad1)
- R4 pad 2: Net-(C7-Pad1) -> Net-(C10-Pad1)
- R5 pad 2: Net-(R5-Pad2) -> Net-(Q1-Pad1)
- R6 pad 1: Net-(R5-Pad2) -> Net-(Q2-Pad3)
- R6 pad 2: GND -> Net-(Q2-Pad1)
- R7 pad 1: GND -> Net-(Q3-Pad3)
- R7 pad 2: Net-(R7-Pad2) -> Net-(Q3-Pad1)
- R8 pad 1: Net-(R7-Pad2) -> Net-(Q4-Pad3)
- R8 pad 2: Net-(R8-Pad2) -> Net-(Q4-Pad1)
- R9 pad 1: Net-(R8-Pad2) -> Net-(C7-Pad2)
- R9 pad 2: Net-(C7-Pad2) -> Net-(R29-Pad2)
- U1 pad 3: Net-(C6-Pad1) -> Net-(R33-Pad1)
- U1 pad 5: Net-(R5-Pad2) -> Net-(R13-Pad2)
- U1 pad 6: Net-(R7-Pad2) -> Net-(R21-Pad2)
- U1 pad 7: Net-(R8-Pad2) -> Net-(R29-Pad2)
Routing:
- net VCC: track 73.7 -> 248.0 mm
- net VDD: track 0.00 -> 116.0 mm
- net Net-(R33-Pad1): track 0.00 -> 113.6 mm
- net GND: track 112.1 -> 22.9 mm, vias 0 -> 6
- net Net-(Q4-Pad1): track 0.00 -> 39.4 mm, vias 0 -> 1
- net Net-(Q3-Pad1): track 0.00 -> 39.4 mm, vias 0 -> 1
- net Net-(Q1-Pad1): track 0.00 -> 39.4 mm, vias 0 -> 1
- net Net-(Q2-Pad1): track 0.00 -> 39.4 mm, vias 0 -> 1
- net Net-(Q1-Pad3): track 50.8 -> 24.2 mm
- net Net-(C7-Pad1): track 33.0 -> 7.94 mm
- net Net-(Q2-Pad3): track 0.00 -> 24.3 mm
- net Net-(Q3-Pad3): track 0.00 -> 24.2 mm
- net Net-(Q4-Pad3): track 0.00 -> 24.2 mm
- net +5V: track 33.6 -> 11.0 mm, vias 2 -> 0
- net Net-(R7-Pad2): track 20.3 -> 0.00 mm
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- added copper zone on B.Cu, net GND
Other:
- board outline added: 94 x 94 mm

Commit message: koniec?
Parts:
- added J10: Conn_02x01, Connector_Molex:Molex_Mini-Fit_Jr_5566-02A_2x01_P4.20mm_Vertical, F.Cu at (116.8, 190.9)
- added J11: Conn_02x01, Connector_Molex:Molex_Mini-Fit_Jr_5566-02A_2x01_P4.20mm_Vertical, F.Cu at (261.6, 149.9)
- added J12: Load +, MountingHole:MountingHole_3.2mm_M3_Pad, F.Cu at (102.9, 116.8)
- added J13: Load -, MountingHole:MountingHole_3.2mm_M3_Pad, F.Cu at (76.2, 119.4)
- added J14: Conn_01x02, Connector_Molex:Molex_Mini-Fit_Jr_5566-02A_2x01_P4.20mm_Vertical, F.Cu at (113.0, 116.8)
- added J3: Conn_01x02, Connector_Molex:Molex_Mini-Fit_Jr_5566-02A_2x01_P4.20mm_Vertical, F.Cu at (203.6, 114.3)
- added J4: Conn_02x01, Connector_Molex:Molex_Mini-Fit_Jr_5566-02A_2x01_P4.20mm_Vertical, F.Cu at (116.8, 137.2)
- added J5: Conn_02x01, Connector_Molex:Molex_Mini-Fit_Jr_5566-02A_2x01_P4.20mm_Vertical, F.Cu at (182.9, 127.0)
- added J6: Conn_02x01, Connector_Molex:Molex_Mini-Fit_Jr_5566-02A_2x01_P4.20mm_Vertical, F.Cu at (116.8, 173.1)
- added J7: Conn_02x01, Connector_Molex:Molex_Mini-Fit_Jr_5566-02A_2x01_P4.20mm_Vertical, F.Cu at (261.6, 132.5)
- added J8: Conn_02x01, Connector_Molex:Molex_Mini-Fit_Jr_5566-02A_2x01_P4.20mm_Vertical, F.Cu at (116.8, 154.9)
- added J9: Conn_02x01, Connector_Molex:Molex_Mini-Fit_Jr_5566-02A_2x01_P4.20mm_Vertical, F.Cu at (182.9, 149.9)
- J1: value Load + -> Ctrl +; footprint Connector_PinHeader_2.54mm:PinHeader_1x01_P2.54mm_Vertical -> MountingHole:MountingHole_3.2mm_M3_Pad
- J2: value Load - -> Ctrl -; footprint Connector_PinHeader_2.54mm:PinHeader_1x01_P2.54mm_Vertical -> MountingHole:MountingHole_3.2mm_M3_Pad
- Q1, Q2, Q3, Q4: footprint Package_TO_SOT_THT:TO-220-3_Vertical -> Package_TO_SOT_THT:TO-220-3_Horizontal_TabDown
- moved R6 144.1 mm to (251.5, 131.1), turned to 270 degrees
- moved R8 144.1 mm to (251.5, 148.8), turned to 270 degrees
- moved Q2 135.0 mm to (246.4, 132.1)
- moved Q4 135.0 mm to (246.4, 149.9)
- moved Q1 81.6 mm to (198.1, 127.0), turned to 270 degrees
- moved Q3 81.6 mm to (198.1, 144.8), turned to 270 degrees
- moved R5 80.5 mm to (193.0, 128.0), turned to 90 degrees
- moved R7 80.5 mm to (193.0, 145.8), turned to 90 degrees
- moved J1 17.0 mm to (63.5, 127.0)
- moved J2 10.8 mm to (63.5, 139.7)
- moved C4 7.62 mm to (66.0, 156.8)
- moved C5 7.62 mm to (62.5, 167.6)
- moved C6 7.62 mm to (67.6, 180.3)
- moved R34 7.62 mm to (67.6, 188.0)
- moved C1 7.62 mm to (61.0, 156.8)
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Connections:
- Q1 pad 1: Net-(Q1-Pad1) -> VDD
- Q1 pad 2: VDD -> Net-(J5-Pad1)
- Q1 pad 3: Net-(Q1-Pad3) -> Net-(J5-Pad2)
- Q2 pad 1: Net-(Q2-Pad1) -> VDD
- Q2 pad 2: VDD -> Net-(J7-Pad1)
- Q2 pad 3: Net-(Q2-Pad3) -> Net-(J7-Pad2)
- Q3 pad 1: Net-(Q3-Pad1) -> VDD
- Q3 pad 2: VDD -> Net-(J9-Pad1)
- Q3 pad 3: Net-(Q3-Pad3) -> Net-(J9-Pad2)
- Q4 pad 1: Net-(Q4-Pad1) -> VDD
- Q4 pad 2: VDD -> Net-(J11-Pad1)
- Q4 pad 3: Net-(Q4-Pad3) -> Net-(J11-Pad2)
- R1 pad 1: Net-(Q1-Pad1) -> Net-(J4-Pad1)
- R13 pad 1: Net-(Q1-Pad3) -> Net-(J4-Pad2)
- R14 pad 1: Net-(Q2-Pad3) -> Net-(J6-Pad2)
- R15 pad 1: Net-(Q3-Pad3) -> Net-(J8-Pad2)
- R16 pad 1: Net-(Q4-Pad3) -> Net-(J10-Pad2)
- R17 pad 1: Net-(Q1-Pad3) -> Net-(J4-Pad2)
- R18 pad 1: Net-(Q2-Pad3) -> Net-(J6-Pad2)
- R19 pad 1: Net-(Q3-Pad3) -> Net-(J8-Pad2)
- R2 pad 1: Net-(Q2-Pad1) -> Net-(J6-Pad1)
- R20 pad 1: Net-(Q4-Pad3) -> Net-(J10-Pad2)
- R3 pad 1: Net-(Q3-Pad1) -> Net-(J8-Pad1)
- R4 pad 1: Net-(Q4-Pad1) -> Net-(J10-Pad1)
- R5 pad 1: Net-(Q1-Pad3) -> Net-(J5-Pad2)
- R5 pad 2: Net-(Q1-Pad1) -> VDD
- R6 pad 1: Net-(Q2-Pad3) -> Net-(J7-Pad2)
- R6 pad 2: Net-(Q2-Pad1) -> VDD
- R7 pad 1: Net-(Q3-Pad3) -> Net-(J9-Pad2)
- R7 pad 2: Net-(Q3-Pad1) -> VDD
- R8 pad 1: Net-(Q4-Pad3) -> Net-(J11-Pad2)
- R8 pad 2: Net-(Q4-Pad1) -> VDD
Routing:
- net GND: track 22.9 -> 163.9 mm, vias 6 -> 10
- net VDD: track 116.0 -> 20.3 mm
- net Net-(Q4-Pad1): track 39.4 -> 0.00 mm, vias 1 -> 0
- net Net-(Q3-Pad1): track 39.4 -> 0.00 mm, vias 1 -> 0
- net Net-(Q1-Pad1): track 39.4 -> 0.00 mm, vias 1 -> 0
- net Net-(Q2-Pad1): track 39.4 -> 0.00 mm, vias 1 -> 0
- net VCC: track 248.0 -> 282.5 mm, vias 0 -> 5
- net Net-(J8-Pad1): track 0.00 -> 31.9 mm
- net Net-(J4-Pad1): track 0.00 -> 31.9 mm
- net Net-(J10-Pad1): track 0.00 -> 31.7 mm
- net Net-(J6-Pad1): track 0.00 -> 31.7 mm
- net Net-(J6-Pad2): track 0.00 -> 27.5 mm
- net Net-(J10-Pad2): track 0.00 -> 27.3 mm
- net Net-(J8-Pad2): track 0.00 -> 26.9 mm
- net Net-(J4-Pad2): track 0.00 -> 26.9 mm
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- added copper zone on B.Cu, net VDD
Other:
- board size 94 x 94 mm -> 210.8 x 94 mm

Commit message: print
Parts:
- added C1: 10u, Capacitor_SMD:C_0805_2012Metric_Pad1.15x1.40mm_HandSolder, B.Cu at (216.2, 71.1)
- added C10: 10n, Capacitor_SMD:C_0805_2012Metric_Pad1.15x1.40mm_HandSolder, B.Cu at (185.7, 92.7)
- added C11: 100n, Capacitor_SMD:C_0805_2012Metric_Pad1.15x1.40mm_HandSolder, B.Cu at (219.4, 109.0)
- added C12: 100n, Capacitor_SMD:C_0805_2012Metric_Pad1.15x1.40mm_HandSolder, B.Cu at (183.8, 109.0)
- added C2: 100n, Capacitor_SMD:C_0805_2012Metric_Pad1.15x1.40mm_HandSolder, B.Cu at (237.2, 109.0)
- added C3: 100n, Capacitor_SMD:C_0805_2012Metric_Pad1.15x1.40mm_HandSolder, B.Cu at (201.6, 109.0)
- added C4: 100n, Capacitor_SMD:C_0805_2012Metric_Pad1.15x1.40mm_HandSolder, B.Cu at (216.2, 76.2)
- added C5: 100n, Capacitor_SMD:C_0805_2012Metric_Pad1.15x1.40mm_HandSolder, B.Cu at (205.4, 72.6)
- added C6: 100n, Capacitor_SMD:C_0805_2012Metric_Pad1.15x1.40mm_HandSolder, B.Cu at (192.7, 77.7)
- added C7: 10n, Capacitor_SMD:C_0805_2012Metric_Pad1.15x1.40mm_HandSolder, B.Cu at (239.1, 92.7)
- added C8: 10n, Capacitor_SMD:C_0805_2012Metric_Pad1.15x1.40mm_HandSolder, B.Cu at (203.5, 92.7)
- added C9: 10n, Capacitor_SMD:C_0805_2012Metric_Pad1.15x1.40mm_HandSolder, B.Cu at (221.3, 92.7)
- added J1: Ctrl +, MountingHole:MountingHole_3.2mm_M3_Pad, F.Cu at (246.1, 73.7)
- added J10: Conn_02x01, Connector_Molex:Molex_Mini-Fit_Jr_5566-02A_2x01_P4.20mm_Vertical, F.Cu at (182.1, 127.0)
- added J12: Load +, MountingHole:MountingHole_3.2mm_M3_Pad, F.Cu at (256.2, 113.0)
- added J13: Load -, MountingHole:MountingHole_3.2mm_M3_Pad, F.Cu at (256.2, 86.4)
- added J14: Conn_01x02, Connector_Molex:Molex_Mini-Fit_Jr_5566-02A_2x01_P4.20mm_Vertical, F.Cu at (256.2, 127.0)
- added J2: Ctrl -, MountingHole:MountingHole_3.2mm_M3_Pad, F.Cu at (233.3, 73.7)
- added J4: Conn_02x01, Connector_Molex:Molex_Mini-Fit_Jr_5566-02A_2x01_P4.20mm_Vertical, F.Cu at (235.9, 127.0)
- added J6: Conn_02x01, Connector_Molex:Molex_Mini-Fit_Jr_5566-02A_2x01_P4.20mm_Vertical, F.Cu at (199.9, 127.0)
- added J8: Conn_02x01, Connector_Molex:Molex_Mini-Fit_Jr_5566-02A_2x01_P4.20mm_Vertical, F.Cu at (218.1, 127.0)
- added R1: 100, Resistor_SMD:R_0805_2012Metric_Pad1.15x1.40mm_HandSolder, B.Cu at (233.6, 96.5)
- added R10: 100, Resistor_SMD:R_0805_2012Metric_Pad1.15x1.40mm_HandSolder, B.Cu at (199.1, 100.6)
- added R11: 100, Resistor_SMD:R_0805_2012Metric_Pad1.15x1.40mm_HandSolder, B.Cu at (216.8, 100.6)
- added R12: 100, Resistor_SMD:R_0805_2012Metric_Pad1.15x1.40mm_HandSolder, B.Cu at (181.3, 100.6)
- added R13: 10k, Resistor_SMD:R_0805_2012Metric_Pad1.15x1.40mm_HandSolder, B.Cu at (243.5, 109.0)
- added R14: 10k, Resistor_SMD:R_0805_2012Metric_Pad1.15x1.40mm_HandSolder, B.Cu at (207.9, 108.8)
- added R15: 10k, Resistor_SMD:R_0805_2012Metric_Pad1.15x1.40mm_HandSolder, B.Cu at (225.7, 109.0)
- added R16: 10k, Resistor_SMD:R_0805_2012Metric_Pad1.15x1.40mm_HandSolder, B.Cu at (190.2, 109.0)
- added R17: 0.1, Resistor_THT:R_Axial_DIN0922_L20.0mm_D9.0mm_P30.48mm_Horizontal, F.Cu at (241.0, 116.8)
- added R18: 0.1, Resistor_THT:R_Axial_DIN0922_L20.0mm_D9.0mm_P30.48mm_Horizontal, F.Cu at (205.4, 116.8)
- added R19: 0.1, Resistor_THT:R_Axial_DIN0922_L20.0mm_D9.0mm_P30.48mm_Horizontal, F.Cu at (223.2, 116.8)
- added R2: 100, Resistor_SMD:R_0805_2012Metric_Pad1.15x1.40mm_HandSolder, B.Cu at (198.0, 96.5)
- added R20: 0.1, Resistor_THT:R_Axial_DIN0922_L20.0mm_D9.0mm_P30.48mm_Horizontal, F.Cu at (187.6, 116.8)
- added R21: 10k, Resistor_SMD:R_0805_2012Metric_Pad1.15x1.40mm_HandSolder, B.Cu at (240.3, 109.0)
- added R22: 10k, Resistor_SMD:R_0805_2012Metric_Pad1.15x1.40mm_HandSolder, B.Cu at (204.8, 109.0)
- added R23: 10k, Resistor_SMD:R_0805_2012Metric_Pad1.15x1.40mm_HandSolder, B.Cu at (222.6, 109.0)
- added R24: 10k, Resistor_SMD:R_0805_2012Metric_Pad1.15x1.40mm_HandSolder, B.Cu at (187.0, 109.0)
- added R25: 10k, Resistor_SMD:R_0805_2012Metric_Pad1.15x1.40mm_HandSolder, B.Cu at (246.7, 109.0)
- added R26: 10k, Resistor_SMD:R_0805_2012Metric_Pad1.15x1.40mm_HandSolder, B.Cu at (211.1, 108.8)
- added R27: 10k, Resistor_SMD:R_0805_2012Metric_Pad1.15x1.40mm_HandSolder, B.Cu at (228.9, 109.0)
- added R28: 10k, Resistor_SMD:R_0805_2012Metric_Pad1.15x1.40mm_HandSolder, B.Cu at (193.3, 109.0)
- added R29: 10k, Resistor_SMD:R_0805_2012Metric_Pad1.15x1.40mm_HandSolder, B.Cu at (246.1, 101.4)
- added R3: 100, Resistor_SMD:R_0805_2012Metric_Pad1.15x1.40mm_HandSolder, B.Cu at (215.8, 96.5)
- added R30: 10k, Resistor_SMD:R_0805_2012Metric_Pad1.15x1.40mm_HandSolder, B.Cu at (210.5, 101.4)
- added R31: 10k, Resistor_SMD:R_0805_2012Metric_Pad1.15x1.40mm_HandSolder, B.Cu at (228.3, 101.4)
- added R32: 10k, Resistor_SMD:R_0805_2012Metric_Pad1.15x1.40mm_HandSolder, B.Cu at (192.7, 101.4)
- added R33: 30k, Resistor_SMD:R_0805_2012Metric_Pad1.15x1.40mm_HandSolder, B.Cu at (185.1, 72.1)
- added R34: 10k, Resistor_SMD:R_0805_2012Metric_Pad1.15x1.40mm_HandSolder, B.Cu at (185.1, 77.7)
- added R4: 100, Resistor_SMD:R_0805_2012Metric_Pad1.15x1.40mm_HandSolder, B.Cu at (180.3, 96.5)
- added R9: 100, Resistor_SMD:R_0805_2012Metric_Pad1.15x1.40mm_HandSolder, B.Cu at (234.6, 100.6)
- added RV1: 10k, Potentiometer_THT:Potentiometer_Alps_RK097_Single_Horizontal, F.Cu at (195.2, 73.7)
- added U1: LM358, Package_SO:SO-8_5.3x6.2mm_P1.27mm, B.Cu at (240.3, 100.3)
- added U2: LM7805_TO220, Package_TO_SOT_THT:TO-220-3_Vertical, F.Cu at (219.4, 71.1)
- added U3: MCP1525-TO, Package_TO_SOT_THT:TO-92_Inline_Wide, F.Cu at (209.2, 71.1)
- added U4: LM358, Package_SO:SO-8_5.3x6.2mm_P1.27mm, B.Cu at (204.8, 100.3)
- added U5: LM358, Package_SO:SO-8_5.3x6.2mm_P1.27mm, B.Cu at (222.6, 100.3)
- added U6: LM358, Package_SO:SO-8_5.3x6.2mm_P1.27mm, B.Cu at (187.0, 100.3)
- moved J11 168.3 mm to (134.6, 260.4)
- moved J5 168.3 mm to (55.9, 237.5)
- moved J7 168.3 mm to (134.6, 243.0)
- moved J9 168.3 mm to (55.9, 260.4)
- moved Q1 168.3 mm to (71.1, 237.5)
- moved Q3 168.3 mm to (71.1, 255.3)
- moved Q4 168.3 mm to (119.4, 260.4)
- moved R6 168.3 mm to (124.5, 241.5)
- moved R8 168.3 mm to (124.5, 259.3)
- moved J3 168.3 mm to (76.6, 224.8)
- moved Q2 168.3 mm to (119.4, 242.6)
- moved R7 168.3 mm to (66.0, 256.3)
- moved R5 168.3 mm to (66.0, 238.5)
- moved R33 116.0 mm to (54.6, 72.1), turned to 90 degrees
- moved R34 111.0 mm to (54.6, 77.7), turned to 270 degrees
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Routing:
- net VCC: track 282.5 -> 565.0 mm, vias 5 -> 10
- net GND: track 163.9 -> 327.8 mm, vias 10 -> 20
- net Net-(R33-Pad1): track 106.0 -> 211.9 mm
- net Net-(J8-Pad1): track 31.9 -> 63.7 mm
- net Net-(J4-Pad1): track 31.9 -> 63.7 mm
- net Net-(J10-Pad1): track 31.7 -> 63.4 mm
- net Net-(J6-Pad1): track 31.7 -> 63.3 mm
- net Net-(J6-Pad2): track 27.5 -> 54.9 mm
- net Net-(J10-Pad2): track 27.3 -> 54.6 mm
- net Net-(J4-Pad2): track 26.9 -> 53.8 mm
- net Net-(J8-Pad2): track 26.9 -> 53.8 mm
- net Net-(R12-Pad2): track 14.4 -> 28.8 mm
- net Net-(R10-Pad2): track 14.4 -> 28.8 mm
- net Net-(R11-Pad2): track 14.4 -> 28.8 mm
- net Net-(R29-Pad2): track 14.4 -> 28.8 mm
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Other:
- board size 210.8 x 94 mm -> 224.5 x 212.1 mm
